Commit message: pulled upstream changes

File: src/jackal_description/urdf/accessories/hdl32_mount.urdf.xacro (robot description, xacro)
@@ -1,2 +1,3 @@
+<<<<<<< Updated upstream
 <robot xmlns:xacro="http://wiki.ros.org/xacro">
   <xacro:include filename="$(find velodyne_description)/urdf/HDL-32E.urdf.xacro" />
@@ -42,2 +43,47 @@
   </xacro:macro>
 </robot>
+=======
+<robot xmlns:xacro="http://wiki.ros.org/xacro">
+  <xacro:include filename="$(find velodyne_description)/urdf/HDL-32E.urdf.xacro" />
+  <xacro:macro name="hdl32e_mount" params="prefix parent_link topic tower *origin">
+    <xacro:if value="${tower}">
+      <link name="${prefix}_hdl32e_mount">
+        <visual>
+          <geometry>
+            <mesh filename="package://jackal_description/meshes/velodyne_tower.stl"/>
+          </geometry>
+          <origin xyz="0 0 0" rpy="0 0 0" />
+          <material name="black" />
+        </visual>
+        <collision>
+          <geometry>
+            <mesh filename="package://jackal_description/meshes/velodyne_tower.stl"/>
+          </geometry>
+          <origin xyz="0 0 0" rpy="0 0 0" />
+        </collision>
+      </link>
+      <joint name="${prefix}_hdl32e_mount_joint" type="fixed">
+        <parent link="${parent_link}" />
+        <child link="${prefix}_hdl32e_mount" />
+        <xacro:insert_block name="origin" />
+      </joint>
+      <!-- Velodyne HDL-32E Macro treats Y-axis as forward in pointcloud -->
+      <xacro:HDL-32E parent="${prefix}_hdl32e_mount" topic="${topic}">
+        <origin xyz="0 0 0.081" rpy="0 0 -1.5707" />
+      </xacro:HDL-32E>
+    </xacro:if>
+    <xacro:unless value="${tower}">
+      <link name="${prefix}_hdl32e_mount"/>
+      <joint name="${prefix}_hdl32e_mount_joint" type="fixed">
+        <parent link="${parent_link}"/>
+        <child link="${prefix}_hdl32e_mount"/>
+        <xacro:insert_block name="origin" />
+      </joint>
+      <!-- Velodyne HDL-32E Macro treats Y-axis as forward in pointcloud -->
+      <xacro:HDL-32E parent="${prefix}_hdl32e_mount" topic="${topic}">
+        <origin xyz="0 0 0" rpy="0 0 -1.5707"/>
+      </xacro:HDL-32E>
+    </xacro:unless>
+  </xacro:macro>
+</robot>
+>>>>>>> Stashed changes

File: src/jackal_description/urdf/accessories/standoffs.urdf.xacro (robot description, xacro)
@@ -1,2 +1,3 @@
+<<<<<<< Updated upstream
 <?xml version="1.0"?>
 <robot xmlns:xacro="http://www.ros.org/wiki/xacro">
@@ -34,2 +35,39 @@
   </xacro:macro>
 </robot>
+=======
+<?xml version="1.0"?>
+<robot xmlns:xacro="http://www.ros.org/wiki/xacro">
+  <!-- Generate a single payload plate standoff. -->
+  <xacro:macro name="standoff" params="name length parent *origin">
+    <link name="${name}">
+      <visual>
+        <origin xyz="0 0 ${length/2}" rpy="0 0 0" />
+        <geometry>
+          <cylinder radius="0.004" length="${length}" />
+        </geometry>
+        <material name="light_grey" />
+      </visual>
+    </link>
+    <joint name="${name}_joint" type="fixed">
+      <xacro:insert_block name="origin" />
+      <parent link="${parent}" />
+      <child link="${name}" />
+    </joint>
+  </xacro:macro>
+  <!-- Generate a set of four standoffs from a payload mount point. -->
+  <xacro:macro name="standoff_box" params="prefix parent height">
+    <xacro:standoff name="${prefix}_standoff0" length="${height}" parent="${parent}">
+      <origin xyz="0.060 0.060 0" rpy="0 0 0"/>
+    </xacro:standoff>
+    <xacro:standoff name="${prefix}_standoff1" length="${height}" parent="${parent}">
+      <origin xyz="0.060 -0.060 0" rpy="0 0 0"/>
+    </xacro:standoff>
+    <xacro:standoff name="${prefix}_standoff2" length="${height}" parent="${parent}">
+      <origin xyz="-0.060 0.060 0" rpy="0 0 0"/>
+    </xacro:standoff>
+    <xacro:standoff name="${prefix}_standoff3" length="${height}" parent="${parent}">
+      <origin xyz="-0.060 -0.060 0" rpy="0 0 0"/>
+    </xacro:standoff>
+  </xacro:macro>
+</robot>
+>>>>>>> Stashed changes

File: src/jackal_description/urdf/accessories/vlp16_mount.urdf.xacro (robot description, xacro)
@@ -1,2 +1,3 @@
+<<<<<<< Updated upstream
 <robot xmlns:xacro="http://wiki.ros.org/xacro">
   <xacro:include filename="$(find velodyne_description)/urdf/VLP-16.urdf.xacro" />
@@ -98,2 +99,103 @@
   </xacro:macro>
 </robot>
+=======
+<robot xmlns:xacro="http://wiki.ros.org/xacro">
+  <xacro:include filename="$(find velodyne_description)/urdf/VLP-16.urdf.xacro" />
+  <xacro:macro name="vlp16_mount" params="prefix parent_link topic tower height:=0.1 *origin">
+    <xacro:if value="${tower}">
+      <link name="${prefix}_vlp16_mount" />
+      <link name="${prefix}_vlp16_plate">
+        <visual>
+          <geometry>
+            <box size="0.1 0.1 0.002" />
+          </geometry>
+          <material name="black" />
+          <origin xyz="0 0 -0.001" rpy="0 0 0" />
+        </visual>
+      </link>
+      <link name="${prefix}_vlp16_leg1">
+        <visual>
+          <geometry>
+            <cylinder length="${height}" radius="0.003" />
+          </geometry>
+          <material name="white">
+            <color rgba="1 1 1 1" />
+          </material>
+          <origin xyz="0 0 ${height/2}" rpy="0 0 0" />
+        </visual>
+      </link>
+      <link name="${prefix}_vlp16_leg2">
+        <visual>
+          <geometry>
+            <cylinder length="${height}" radius="0.003" />
+          </geometry>
+          <material name="white">
+            <color rgba="1 1 1 1" />
+          </material>
+          <origin xyz="0 0 ${height/2}" rpy="0 0 0" />
+        </visual>
+      </link>
+      <link name="${prefix}_vlp16_leg3">
+        <visual>
+          <geometry>
+            <cylinder length="${height}" radius="0.003" />
+          </geometry>
+          <material name="white">
+            <color rgba="1 1 1 1" />
+          </material>
+          <origin xyz="0 0 ${height/2}" rpy="0 0 0" />
+        </visual>
+      </link>
+      <link name="${prefix}_vlp16_leg4">
+        <visual>
+          <geometry>
+            <cylinder length="${height}" radius="0.003" />
+          </geometry>
+          <material name="white">
+            <color rgba="1 1 1 1" />
+          </material>
+          <origin xyz="0 0 ${height/2}" rpy="0 0 0" />
+        </visual>
+      </link>
+      <joint name="${prefix}_vlp16_mount_joint" type="fixed">
+        <parent link="${parent_link}" />
+        <child link="${prefix}_vlp16_mount" />
+        <xacro:insert_block name="origin" />
+      </joint>
+      <joint name="${prefix}_vlp16_leg1_joint" type="fixed">
+        <parent link="${prefix}_vlp16_mount" />
+        <child link="${prefix}_vlp16_leg1" />
+        <origin xyz="0.05 0.05 0" rpy="0 0 0" />
+      </joint>
+      <joint name="${prefix}_vlp16_leg2_joint" type="fixed">
+        <parent link="${prefix}_vlp16_mount" />
+        <child link="${prefix}_vlp16_leg2" />
+        <origin xyz="0.05 -0.05 0" rpy="0 0 0" />
+      </joint>
+      <joint name="${prefix}_vlp16_leg3_joint" type="fixed">
+        <parent link="${prefix}_vlp16_mount" />
+        <child link="${prefix}_vlp16_leg3" />
+        <origin xyz="-0.05 0.05 0" rpy="0 0 0" />
+      </joint>
+      <joint name="${prefix}_vlp16_leg4_joint" type="fixed">
+        <parent link="${prefix}_vlp16_mount" />
+        <child link="${prefix}_vlp16_leg4" />
+        <origin xyz="-0.05 -0.05 0" rpy="0 0 0" />
+      </joint>
+      <joint name="${prefix}_vlp16_plate_joint" type="fixed">
+        <parent link="${prefix}_vlp16_mount" />
+        <child link="${prefix}_vlp16_plate" />
+        <origin xyz="0 0 ${height}" rpy="0 0 0" />
+      </joint>
+      <xacro:VLP-16 parent="${prefix}_vlp16_plate" topic="${topic}">
+        <origin xyz="0 0 0" rpy="0 0 0" />
+      </xacro:VLP-16>
+    </xacro:if>
+    <xacro:unless value="${tower}">
+      <xacro:VLP-16 parent="${parent_link}" topic="${topic}">
+        <xacro:insert_block name="origin" />
+      </xacro:VLP-16>
+    </xacro:unless>
+  </xacro:macro>
+</robot>
+>>>>>>> Stashed changes
